File: lora.sch (KiCad schematic (older format))
At the start: 55 parts, among them J1 Conn_01x02, J10 Conn, J11 Conn_Coaxial, J2 Humidity, J3 Temp, J4 Programming_Jumper, J5 Temp, J6 VDD, J7 GPS, J8 SIM800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

Commit message: some more structure and 2 additonal layers, first board outlines....
Parts:
- added C? (x2): dnp, Capacitor_SMD:C_0603_1608Metric, symbol Device:C_Small
- added L?: 0R, Resistor_SMD:R_0603_1608Metric, symbol Device:L_Small
- C1, C2: footprint Capacitor_SMD:C_0805_2012Metric -> Capacitor_SMD:C_1206_3216Metric; LCSC C15850 -> C13585
Connections:
- net GND: now also C?.1, C?.1
- net at U4.9 (ANT): now also C?.2, L?.1; no longer J11.1 (In)
- new net: C?.2, J11.1 (In), L?.2
Other:
- note added: "Ferit zu Störunterdrückung."
- note removed: "SMA or just a\nsimple short wire"
- moved on the sheet: C9, J11, R13, U4
Changed lines of the file:
@@
 L RF_Module:RFM95W-868S2 U4
 U 1 1 5FAAB373
-P 9775 3950
-F 0 "U4" H 10000 3400 50  0000 C CNN
-F 1 "RFM95W-868S2" H 9375 4425 50  0000 C CNN
-F 2 "RF_Module:HOPERF_RFM9XW_SMD" H 6475 5600 50  0001 C CNN
-F 3 "https://www.hoperf.com/data/upload/portal/20181127/5bfcbea20e9ef.pdf" H 6475 5600 50  0001 C CNN
-	1    9775 3950
+P 9050 3975
+F 0 "U4" H 9275 3425 50  0000 C CNN
+F 1 "RFM95W-868S2" H 8650 4450 50  0000 C CNN
+F 2 "RF_Module:HOPERF_RFM9XW_SMD" H 5750 5625 50  0001 C CNN
+F 3 "https://www.hoperf.com/data/upload/portal/20181127/5bfcbea20e9ef.pdf" H 5750 5625 50  0001 C CNN
+	1    9050 3975
 	1    0    0    -1
 $EndComp
@@
 L power:VDD #PWR0104
 U 1 1 5FAC50BA
-P 9775 3450
-F 0 "#PWR0104" H 9775 3300 50  0001 C CNN
-F 1 "VDD" H 9790 3623 50  0000 C CNN
-F 2 "" H 9775 3450 50  0001 C CNN
-F 3 "" H 9775 3450 50  0001 C CNN
-	1    9775 3450
+P 9050 3475
+F 0 "#PWR0104" H 9050 3325 50  0001 C CNN
+F 1 "VDD" H 9065 3648 50  0000 C CNN
+F 2 "" H 9050 3475 50  0001 C CNN
+F 3 "" H 9050 3475 50  0001 C CNN
+	1    9050 3475
 	1    0    0    -1
 $EndComp
@@
 L power:GND #PWR0106
 U 1 1 5FAC6294
-P 9875 4550
-F 0 "#PWR0106" H 9875 4300 50  0001 C CNN
-F 1 "GND" H 9880 4377 50  0000 C CNN
-F 2 "" H 9875 4550 50  0001 C CNN
-F 3 "" H 9875 4550 50  0001 C CNN
-	1    9875 4550
-	1    0    0    -1
-$EndComp
-Wire Wire Line
-	9675 4550 9775 4550
-Connection ~ 9875 4550
-Connection ~ 9775 4550
-Wire Wire Line
-	9775 4550 9875 4550
+P 9150 4575
+F 0 "#PWR0106" H 9150 4325 50  0001 C CNN
+F 1 "GND" H 9155 4402 50  0000 C CNN
+F 2 "" H 9150 4575 50  0001 C CNN
+F 3 "" H 9150 4575 50  0001 C CNN
+	1    9150 4575
+	1    0    0    -1
+$EndComp
+Wire Wire Line
+	8950 4575 9050 4575
+Connection ~ 9150 4575
+Connection ~ 9050 4575
+Wire Wire Line
+	9050 4575 9150 4575
 $Comp
 L power:GND #PWR0107
@@
 L power:GND #PWR0124
 U 1 1 5FB31B49
-P 10075 3250
-F 0 "#PWR0124" H 10075 3000 50  0001 C CNN
-F 1 "GND" H 10080 3077 50  0000 C CNN
-F 2 "" H 10075 3250 50  0001 C CNN
-F 3 "" H 10075 3250 50  0001 C CNN
-	1    10075 3250
+P 9350 3275
+F 0 "#PWR0124" H 9350 3025 50  0001 C CNN
+F 1 "GND" H 9355 3102 50  0000 C CNN
+F 2 "" H 9350 3275 50  0001 C CNN
+F 3 "" H 9350 3275 50  0001 C CNN
+	1    9350 3275
 	1    0    0    -1
 $EndComp
@@
 L power:VDD #PWR0125
 U 1 1 5FB31B4F
-P 10075 3050
-F 0 "#PWR0125" H 10075 2900 50  0001 C CNN
-F 1 "VDD" H 10090 3223 50  0000 C CNN
-F 2 "" H 10075 3050 50  0001 C CNN
-F 3 "" H 10075 3050 50  0001 C CNN
-	1    10075 3050
+P 9350 3075
+F 0 "#PWR0125" H 9350 2925 50  0001 C CNN
+F 1 "VDD" H 9365 3248 50  0000 C CNN
+F 2 "" H 9350 3075 50  0001 C CNN
+F 3 "" H 9350 3075 50  0001 C CNN
+	1    9350 3075
 	1    0    0    -1
 $EndComp
@@
 L Device:C_Small C9
 U 1 1 5FB31B55
-P 10075 3150
-F 0 "C9" H 9983 3104 50  0000 R CNN
-F 1 "100n" H 9983 3195 50  0000 R CNN
-F 2 "Capacitor_SMD:C_0603_1608Metric" H 10075 3150 50  0001 C CNN
-F 3 "~" H 10075 3150 50  0001 C CNN
-F 4 "C14663" H 10075 3150 50  0001 C CNN "LCSC"
-	1    10075 3150
+P 9350 3175
+F 0 "C9" H 9258 3129 50  0000 R CNN
+F 1 "100n" H 9258 3220 50  0000 R CNN
+F 2 "Capacitor_SMD:C_0603_1608Metric" H 9350 3175 50  0001 C CNN
+F 3 "~" H 9350 3175 50  0001 C CNN
+F 4 "C14663" H 9350 3175 50  0001 C CNN "LCSC"
+	1    9350 3175
 	-1   0    0    1
 $EndComp
@@
 Text GLabel 9700 5900 0    50   Input ~ 0
 UART1_TX
-Text GLabel 9275 3950 0    50   Input ~ 0
+Text GLabel 8550 3975 0    50   Input ~ 0
 SPI_CS
-Text GLabel 9275 3850 0    50   Input ~ 0
+Text GLabel 8550 3875 0    50   Input ~ 0
 SPI_MISO
-Text GLabel 9275 3750 0    50   Input ~ 0
+Text GLabel 8550 3775 0    50   Input ~ 0
 SPI_MOSI
-Text GLabel 9275 3650 0    50   Input ~ 0
+Text GLabel 8550 3675 0    50   Input ~ 0
 SPI_SCK
-Text GLabel 8800 4150 0    50   Input ~ 0
+Text GLabel 8400 4175 0    50   Input ~ 0
 RFM_RST
-Text GLabel 10275 4350 2    50   Input ~ 0
+Text GLabel 9550 4375 2    50   Input ~ 0
 RFM_DIO0
-Text Notes 9100 3400 0    50   ~ 0
+Text Notes 8375 3425 0    50   ~ 0
 1.8V - 3.9V
 $Comp
@@
 L Device:R_Small R13
 U 1 1 5FB148B9
-P 8800 4275
-F 0 "R13" V 8700 4300 50  0000 C CNN
-F 1 "10k" V 8905 4275 50  0000 C CNN
-F 2 "Capacitor_SMD:C_0603_1608Metric" H 8800 4275 50  0001 C CNN
-F 3 "~" H 8800 4275 50  0001 C CNN
-F 4 "C25804" H 8800 4275 50  0001 C CNN "LCSC"
-	1    8800 4275
+P 8400 4300
+F 0 "R13" V 8300 4325 50  0000 C CNN
+F 1 "10k" V 8505 4300 50  0000 C CNN
+F 2 "Capacitor_SMD:C_0603_1608Metric" H 8400 4300 50  0001 C CNN
+F 3 "~" H 8400 4300 50  0001 C CNN
+F 4 "C25804" H 8400 4300 50  0001 C CNN "LCSC"
+	1    8400 4300
 	1    0    0    -1
 $EndComp
@@
 L power:GND #PWR0135
 U 1 1 5FB153E6
-P 8800 4375
-F 0 "#PWR0135" H 8800 4125 50  0001 C CNN
-F 1 "GND" H 8805 4202 50  0000 C CNN
-F 2 "" H 8800 4375 50  0001 C CNN
-F 3 "" H 8800 4375 50  0001 C CNN
-	1    8800 4375
-	1    0    0    -1
-$EndComp
-Wire Wire Line
-	9275 4150 8800 4150
-Wire Wire Line
-	8800 4150 8800 4175
+P 8400 4400
+F 0 "#PWR0135" H 8400 4150 50  0001 C CNN
+F 1 "GND" H 8405 4227 50  0000 C CNN
+F 2 "" H 8400 4400 50  0001 C CNN
+F 3 "" H 8400 4400 50  0001 C CNN
+	1    8400 4400
+	1    0    0    -1
+$EndComp
+Wire Wire Line
+	8400 4175 8400 4200
 $Comp
 L Connector_Generic:Conn_01x03 J5
@@
 F 0 "C1" H 958 1154 50  0000 R CNN
 F 1 "10u" H 958 1245 50  0000 R CNN
-F 2 "Capacitor_SMD:C_0805_2012Metric" H 1050 1200 50  0001 C CNN
+F 2 "Capacitor_SMD:C_1206_3216Metric" H 1050 1200 50  0001 C CNN
 F 3 "~" H 1050 1200 50  0001 C CNN
-F 4 "C15850" H 1050 1200 50  0001 C CNN "LCSC"
+F 4 "C13585" H 1050 1200 50  0001 C CNN "LCSC"
 	1    1050 1200
 	-1   0    0    1
@@
 F 0 "C2" H 1308 1154 50  0000 R CNN
 F 1 "10u" H 1308 1245 50  0000 R CNN
-F 2 "Capacitor_SMD:C_0805_2012Metric" H 1400 1200 50  0001 C CNN
+F 2 "Capacitor_SMD:C_1206_3216Metric" H 1400 1200 50  0001 C CNN
 F 3 "~" H 1400 1200 50  0001 C CNN
-F 4 "C15850" H 1400 1200 50  0001 C CNN "LCSC"
+F 4 "C13585" H 1400 1200 50  0001 C CNN "LCSC"
 	1    1400 1200
 	-1   0    0    1
@@
 Wire Notes Line
 	475  6050 6975 6050
-NoConn ~ 10275 4250
-NoConn ~ 10275 4150
-NoConn ~ 10275 4050
-NoConn ~ 10275 3950
-NoConn ~ 10275 3850
+NoConn ~ 9550 4275
+NoConn ~ 9550 4175
+NoConn ~ 9550 4075
+NoConn ~ 9550 3975
+NoConn ~ 9550 3875
 $Comp
 L Device:R_Small R17
@@
 L Connector:Conn_Coaxial J11
 U 1 1 5FC31EE2
-P 10475 3650
-F 0 "J11" H 10575 3625 50  0000 L CNN
-F 1 "Conn_Coaxial" H 10575 3534 50  0000 L CNN
-F 2 "Connector_Coaxial:SMA_Amphenol_132134_Vertical" H 10475 3650 50  0001 C CNN
-F 3 " ~" H 10475 3650 50  0001 C CNN
-	1    10475 3650
+P 10250 3675
+F 0 "J11" H 10350 3650 50  0000 L CNN
+F 1 "Conn_Coaxial" V 10400 3725 50  0000 L CNN
+F 2 "Connector_Coaxial:SMA_Amphenol_132134_Vertical" H 10250 3675 50  0001 C CNN
+F 3 " ~" H 10250 3675 50  0001 C CNN
+	1    10250 3675
 	1    0    0    -1
 $EndComp
@@
 L power:GND #PWR0146
 U 1 1 5FC3451D
-P 10475 3850
-F 0 "#PWR0146" H 10475 3600 50  0001 C CNN
-F 1 "GND" H 10480 3677 50  0000 C CNN
-F 2 "" H 10475 3850 50  0001 C CNN
-F 3 "" H 10475 3850 50  0001 C CNN
-	1    10475 3850
-	1    0    0    -1
-$EndComp
-Text Notes 10275 3500 0    50   ~ 0
-SMA or just a\nsimple short wire
+P 10250 3875
+F 0 "#PWR0146" H 10250 3625 50  0001 C CNN
+F 1 "GND" H 10255 3702 50  0000 C CNN
+F 2 "" H 10250 3875 50  0001 C CNN
+F 3 "" H 10250 3875 50  0001 C CNN
+	1    10250 3875
+	1    0    0    -1
+$EndComp
 $Comp
 L Device:Crystal Y1
@@
 Text Notes 4225 2675 0    50   ~ 0
 Shall consume \nless then 100nA
+$Comp
+L Device:C_Small C?
+U 1 1 5FC2AFEC
+P 9875 3775
+F 0 "C?" H 9783 3729 50  0000 R CNN
+F 1 "dnp" H 9783 3820 50  0000 R CNN
+F 2 "Capacitor_SMD:C_0603_1608Metric" H 9875 3775 50  0001 C CNN
+F 3 "~" H 9875 3775 50  0001 C CNN
+F 4 "" H 9875 3775 50  0001 C CNN "LCSC"
+	1    9875 3775
+	-1   0    0    1
+$EndComp
+Wire Wire Line
+	8550 4175 8400 4175
+$Comp
+L Device:L_Small L?
+U 1 1 5FC42B81
+P 9775 3675
+F 0 "L?" V 9960 3675 50  0000 C CNN
+F 1 "0R" V 9869 3675 50  0000 C CNN
+F 2 "Resistor_SMD:R_0603_1608Metric" H 9775 3675 50  0001 C CNN
+F 3 "~" H 9775 3675 50  0001 C CNN
+F 4 "C21189" V 9775 3675 50  0001 C CNN "LCSC"
+	1    9775 3675
+	0    -1   -1   0
+$EndComp
+$Comp
+L Device:C_Small C?
+U 1 1 5FC4504E
+P 9675 3775
+F 0 "C?" H 9850 3800 50  0000 R CNN
+F 1 "dnp" H 9875 3725 50  0000 R CNN
+F 2 "Capacitor_SMD:C_0603_1608Metric" H 9675 3775 50  0001 C CNN
+F 3 "~" H 9675 3775 50  0001 C CNN
+F 4 "" H 9675 3775 50  0001 C CNN "LCSC"
+	1    9675 3775
+	-1   0    0    1
+$EndComp
+Wire Wire Line
+	9550 3675 9675 3675
+Connection ~ 9675 3675
+Wire Wire Line
+	9875 3675 10050 3675
+Connection ~ 9875 3675
+Wire Wire Line
+	10250 3875 9875 3875
+Connection ~ 10250 3875
+Wire Wire Line
+	9875 3875 9675 3875
+Connection ~ 9875 3875
+Text Notes -850 1200 0    50   ~ 0
+Ferit  zu Störunterdrückung.
 $EndSCHEMATC
