File: pcb/lora.kicad_sch (KiCad schematic)
At the start: 91 parts, among them J1 Conn_01x04, J11 Conn_Coaxial, J2 5V, J3 Conn_01x06, J4 USB_C_Receptacle_USB2.0, J5 Temp, J6 VDD, J7 UART, J8 Conn_01x04, Q1 AO3401A, Q2 AO3401A, Q3 AO3401A, Q5 AO3401A, SW1 RESET, SW2 PJ, SW3 K3-1296S-E1, U1 ME2108C50M5G, U2 ESP32-WROOM-32D, U3 2460, U4 RFM95W-868S2, U5 SCT2400, U6 CH340E

Commit message: more silkscreen text
Parts:
- C4: value 47u -> 22u; LCSC C403725 -> C342620
- R25: LCSC (none) -> C22935
- R26, R27: LCSC (none) -> C23067
- U2: LCSC (none) -> C473012
Other:
- note added: "5 - 25V"
Changed lines of the file:
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@@
     (effects (font (size 1.27 1.27)) (justify left bottom))
   )
+  (text "5 - 25V" (at 54.356 76.708 0)
+    (effects (font (size 1.27 1.27)) (justify left bottom))
+  )
   (text "floating for flashing" (at 172.72 85.09 0)
     (effects (font (size 1.27 1.27)) (justify left bottom))
@@
       (effects (font (size 1.27 1.27)) hide)
     )
+    (property "LCSC" "C473012" (id 4) (at 155.575 109.855 0)
+      (effects (font (size 1.27 1.27)) hide)
+    )
     (pin "1")
     (pin "10")
@@
       (effects (font (size 1.27 1.27)) hide)
     )
-    (property "LCSC" "" (id 4) (at 83.058 152.654 0)
+    (property "LCSC" "C23067" (id 4) (at 83.058 152.654 0)
       (effects (font (size 1.27 1.27)) hide)
     )
@@
       (effects (font (size 1.27 1.27)) hide)
     )
-    (property "LCSC" "" (id 4) (at 55.626 188.214 0)
+    (property "LCSC" "C22935" (id 4) (at 55.626 188.214 0)
       (effects (font (size 1.27 1.27)) hide)
     )
@@
       (effects (font (size 1.27 1.27)) hide)
     )
-    (property "LCSC" "" (id 4) (at 83.312 155.194 0)
+    (property "LCSC" "C23067" (id 4) (at 83.312 155.194 0)
       (effects (font (size 1.27 1.27)) hide)
     )
@@
       (effects (font (size 1.27 1.27)) (justify left))
     )
-    (property "Value" "47u" (id 1) (at 20.828 30.353 0)
+    (property "Value" "22u" (id 1) (at 20.828 30.353 0)
       (effects (font (size 1.27 1.27)) (justify left))
     )
@@
       (effects (font (size 1.27 1.27)) hide)
     )
-    (property "LCSC" "C403725" (id 4) (at 22.606 26.289 0)
+    (property "LCSC" "C342620" (id 4) (at 22.606 26.289 0)
       (effects (font (size 1.27 1.27)) hide)
     )
@@
     )
     (path "/a7c486da-70fc-43e8-9b1b-356c5879de2f"
-      (reference "C4") (unit 1) (value "47u") (footprint "Capacitor_SMD:C_1206_3216Metric")
+      (reference "C4") (unit 1) (value "22u") (footprint "Capacitor_SMD:C_1206_3216Metric")
     )
     (path "/00000000-0000-0000-0000-00005fb2a8d7"

Commit message: changed a capacity
Parts:
- C3: value 47u -> 10u; footprint Capacitor_SMD:C_1210_3225Metric -> Capacitor_SMD:C_0805_2012Metric; LCSC C77101 -> C440198
Changed lines of the file:
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@@
       (effects (font (size 1.27 1.27)) (justify right))
     )
-    (property "Value" "47u" (id 1) (at 263.7028 49.657 0)
-      (effects (font (size 1.27 1.27)) (justify right))
-    )
-    (property "Footprint" "Capacitor_SMD:C_1210_3225Metric" (id 2) (at 261.366 48.514 0)
+    (property "Value" "10u" (id 1) (at 263.7028 49.657 0)
+      (effects (font (size 1.27 1.27)) (justify right))
+    )
+    (property "Footprint" "Capacitor_SMD:C_0805_2012Metric" (id 2) (at 261.366 48.514 0)
       (effects (font (size 1.27 1.27)) hide)
     )
@@
       (effects (font (size 1.27 1.27)) hide)
     )
-    (property "LCSC" "C77101" (id 4) (at 261.366 48.514 0)
+    (property "LCSC" "C440198" (id 4) (at 261.366 48.514 0)
       (effects (font (size 1.27 1.27)) hide)
     )
@@
     )
     (path "/8ee164e2-ecd6-40c2-9fb8-70638f6591db"
-      (reference "C3") (unit 1) (value "47u") (footprint "Capacitor_SMD:C_1210_3225Metric")
+      (reference "C3") (unit 1) (value "10u") (footprint "Capacitor_SMD:C_0805_2012Metric")
     )
     (path "/a7c486da-70fc-43e8-9b1b-356c5879de2f"

Commit message: updated readme
Parts:
- R1, R11, R13, R17, R2, R20, R23, R24, R3, R4, R5, R6, R9: footprint Capacitor_SMD:C_0603_1608Metric -> Resistor_SMD:R_0603_1608Metric
Changed lines of the file:
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@@
     (property "Reference" "R3" (id 0) (at 113.919 76.2 90))
     (property "Value" "10k" (id 1) (at 114.554 70.993 90))
-    (property "Footprint" "Capacitor_SMD:C_0603_1608Metric" (id 2) (at 114.554 73.66 0)
+    (property "Footprint" "Resistor_SMD:R_0603_1608Metric" (id 2) (at 114.554 73.66 0)
       (effects (font (size 1.27 1.27)) hide)
     )
@@
     (property "Reference" "R11" (id 0) (at 222.0214 22.6822 90))
     (property "Value" "10k" (id 1) (at 227.2284 23.3172 90))
-    (property "Footprint" "Capacitor_SMD:C_0603_1608Metric" (id 2) (at 224.5614 23.3172 0)
+    (property "Footprint" "Resistor_SMD:R_0603_1608Metric" (id 2) (at 224.5614 23.3172 0)
       (effects (font (size 1.27 1.27)) hide)
     )
@@
     (property "Reference" "R9" (id 0) (at 151.2824 164.465 90))
     (property "Value" "10k" (id 1) (at 156.4894 165.1 90))
-    (property "Footprint" "Capacitor_SMD:C_0603_1608Metric" (id 2) (at 153.8224 165.1 0)
+    (property "Footprint" "Resistor_SMD:R_0603_1608Metric" (id 2) (at 153.8224 165.1 0)
       (effects (font (size 1.27 1.27)) hide)
     )
@@
     (property "Reference" "R4" (id 0) (at 113.665 50.038 90))
     (property "Value" "10k" (id 1) (at 114.3 44.831 90))
-    (property "Footprint" "Capacitor_SMD:C_0603_1608Metric" (id 2) (at 114.3 47.498 0)
+    (property "Footprint" "Resistor_SMD:R_0603_1608Metric" (id 2) (at 114.3 47.498 0)
       (effects (font (size 1.27 1.27)) hide)
     )
@@
     (property "Reference" "R5" (id 0) (at 208.915 86.36 90))
     (property "Value" "10k" (id 1) (at 209.55 82.55 90))
-    (property "Footprint" "Capacitor_SMD:C_0603_1608Metric" (id 2) (at 210.82 86.995 0)
+    (property "Footprint" "Resistor_SMD:R_0603_1608Metric" (id 2) (at 210.82 86.995 0)
       (effects (font (size 1.27 1.27)) hide)
     )
@@
     (property "Reference" "R6" (id 0) (at 213.995 85.725 90))
     (property "Value" "10k" (id 1) (at 211.455 75.565 90))
-    (property "Footprint" "Capacitor_SMD:C_0603_1608Metric" (id 2) (at 212.725 80.645 0)
+    (property "Footprint" "Resistor_SMD:R_0603_1608Metric" (id 2) (at 212.725 80.645 0)
       (effects (font (size 1.27 1.27)) hide)
     )
@@
     (property "Reference" "R13" (id 0) (at 216.535 80.645 90))
     (property "Value" "10k" (id 1) (at 213.995 71.12 90))
-    (property "Footprint" "Capacitor_SMD:C_0603_1608Metric" (id 2) (at 215.265 75.565 0)
+    (property "Footprint" "Resistor_SMD:R_0603_1608Metric" (id 2) (at 215.265 75.565 0)
       (effects (font (size 1.27 1.27)) hide)
     )
@@
     (property "Reference" "R17" (id 0) (at 222.25 71.12 90))
     (property "Value" "10k" (id 1) (at 220.472 70.485 90))
-    (property "Footprint" "Capacitor_SMD:C_0603_1608Metric" (id 2) (at 217.805 70.485 0)
+    (property "Footprint" "Resistor_SMD:R_0603_1608Metric" (id 2) (at 217.805 70.485 0)
       (effects (font (size 1.27 1.27)) hide)
     )
@@
     (property "Reference" "R20" (id 0) (at 34.8234 96.0882 90))
     (property "Value" "4k7" (id 1) (at 36.576 100.965 90))
-    (property "Footprint" "Capacitor_SMD:C_0603_1608Metric" (id 2) (at 36.576 98.298 0)
+    (property "Footprint" "Resistor_SMD:R_0603_1608Metric" (id 2) (at 36.576 98.298 0)
       (effects (font (size 1.27 1.27)) hide)
     )
@@
     (property "Reference" "R2" (id 0) (at 213.36 107.95 90))
     (property "Value" "10k" (id 1) (at 213.995 104.14 90))
-    (property "Footprint" "Capacitor_SMD:C_0603_1608Metric" (id 2) (at 215.265 108.585 0)
+    (property "Footprint" "Resistor_SMD:R_0603_1608Metric" (id 2) (at 215.265 108.585 0)
       (effects (font (size 1.27 1.27)) hide)
     )
@@
     (property "Reference" "R24" (id 0) (at 105.791 101.727 90))
     (property "Value" "1k" (id 1) (at 102.235 101.854 90))
-    (property "Footprint" "Capacitor_SMD:C_0603_1608Metric" (id 2) (at 103.251 103.632 0)
+    (property "Footprint" "Resistor_SMD:R_0603_1608Metric" (id 2) (at 103.251 103.632 0)
       (effects (font (size 1.27 1.27)) hide)
     )
@@
       (effects (font (size 1.27 1.27) italic) (justify left) hide)
     )
-    (property "Datasheet" "LV2842XLVDDCR" (id 3) (at 51.562 17.399 0)
+    (property "Datasheet" "" (id 3) (at 51.562 17.399 0)
       (effects (font (size 1.27 1.27)) hide)
     )
@@
     (property "Reference" "R1" (id 0) (at 185.928 142.113 90))
     (property "Value" "1k" (id 1) (at 191.135 142.748 90))
-    (property "Footprint" "Capacitor_SMD:C_0603_1608Metric" (id 2) (at 188.468 142.748 0)
+    (property "Footprint" "Resistor_SMD:R_0603_1608Metric" (id 2) (at 188.468 142.748 0)
       (effects (font (size 1.27 1.27)) hide)
     )
@@
     (property "Reference" "R23" (id 0) (at 98.679 110.1852 90))
     (property "Value" "1k" (id 1) (at 97.2312 108.1786 90))
-    (property "Footprint" "Capacitor_SMD:C_0603_1608Metric" (id 2) (at 99.187 106.172 0)
+    (property "Footprint" "Resistor_SMD:R_0603_1608Metric" (id 2) (at 99.187 106.172 0)
       (effects (font (size 1.27 1.27)) hide)
     )
@@
     )
     (path "/e563a71b-5c2b-47a4-be59-4a8b10659a28"
-      (reference "R1") (unit 1) (value "1k") (footprint "Capacitor_SMD:C_0603_1608Metric")
+      (reference "R1") (unit 1) (value "1k") (footprint "Resistor_SMD:R_0603_1608Metric")
     )
     (path "/00000000-0000-0000-0000-00006173cdbc"
-      (reference "R2") (unit 1) (value "10k") (footprint "Capacitor_SMD:C_0603_1608Metric")
+      (reference "R2") (unit 1) (value "10k") (footprint "Resistor_SMD:R_0603_1608Metric")
     )
     (path "/00000000-0000-0000-0000-00005fb032ee"
-      (reference "R3") (unit 1) (value "10k") (footprint "Capacitor_SMD:C_0603_1608Metric")
+      (reference "R3") (unit 1) (value "10k") (footprint "Resistor_SMD:R_0603_1608Metric")
     )
     (path "/00000000-0000-0000-0000-0000613dd3f0"
-      (reference "R4") (unit 1) (value "10k") (footprint "Capacitor_SMD:C_0603_1608Metric")
+      (reference "R4") (unit 1) (value "10k") (footprint "Resistor_SMD:R_0603_1608Metric")
     )
     (path "/00000000-0000-0000-0000-0000613e0914"
-      (reference "R5") (unit 1) (value "10k") (footprint "Capacitor_SMD:C_0603_1608Metric")
+      (reference "R5") (unit 1) (value "10k") (footprint "Resistor_SMD:R_0603_1608Metric")
     )
     (path "/00000000-0000-0000-0000-0000613e1a6b"
-      (reference "R6") (unit 1) (value "10k") (footprint "Capacitor_SMD:C_0603_1608Metric")
+      (reference "R6") (unit 1) (value "10k") (footprint "Resistor_SMD:R_0603_1608Metric")
     )
     (path "/00000000-0000-0000-0000-00005fab81d2"
@@
     )
     (path "/00000000-0000-0000-0000-00005fb418a5"
-      (reference "R9") (unit 1) (value "10k") (footprint "Capacitor_SMD:C_0603_1608Metric")
+      (reference "R9") (unit 1) (value "10k") (footprint "Resistor_SMD:R_0603_1608Metric")
     )
     (path "/00000000-0000-0000-0000-00005fb418b5"
@@
     )
     (path "/00000000-0000-0000-0000-00005fb1dc2c"
-      (reference "R11") (unit 1) (value "10k") (footprint "Capacitor_SMD:C_0603_1608Metric")
+      (reference "R11") (unit 1) (value "10k") (footprint "Resistor_SMD:R_0603_1608Metric")
     )
     (path "/00000000-0000-0000-0000-00005fb1fbf3"
@@
     )
     (path "/00000000-0000-0000-0000-0000613e1cfc"
-      (reference "R13") (unit 1) (value "10k") (footprint "Capacitor_SMD:C_0603_1608Metric")
+      (reference "R13") (unit 1) (value "10k") (footprint "Resistor_SMD:R_0603_1608Metric")
     )
     (path "/ed6b0719-fbd0-4f4c-8787-dd22a8f13adb"
@@
     )
     (path "/00000000-0000-0000-0000-0000613e1fd9"
-      (reference "R17") (unit 1) (value "10k") (footprint "Capacitor_SMD:C_0603_1608Metric")
+      (reference "R17") (unit 1) (value "10k") (footprint "Resistor_SMD:R_0603_1608Metric")
     )
     (path "/4efe1fe8-d248-4230-829d-d43d13736911"
@@
     )
     (path "/00000000-0000-0000-0000-0000614025b8"
-      (reference "R20") (unit 1) (value "4k7") (footprint "Capacitor_SMD:C_0603_1608Metric")
+      (reference "R20") (unit 1) (value "4k7") (footprint "Resistor_SMD:R_0603_1608Metric")
     )
     (path "/99e8ee9b-566b-429f-9c69-d2a9a81e6a1e"
@@
     )
     (path "/f9f61b80-9c7e-4617-936a-eb2a1bd6d588"
-      (reference "R23") (unit 1) (value "1k") (footprint "Capacitor_SMD:C_0603_1608Metric")
+      (reference "R23") (unit 1) (value "1k") (footprint "Resistor_SMD:R_0603_1608Metric")
     )
     (path "/407c8f2a-3a09-435d-b3d0-5876070a2177"
-      (reference "R24") (unit 1) (value "1k") (footprint "Capacitor_SMD:C_0603_1608Metric")
+      (reference "R24") (unit 1) (value "1k") (footprint "Resistor_SMD:R_0603_1608Metric")
     )
     (path "/317cd803-1d55-4d2e-bd68-dff7f92e8364"
